File: PWR.kicad_sch (KiCad schematic)
At the start: 5 parts, among them U8 SE5218

Commit message: Created Version 1.0
Refactored board with tipps after coaching
Parts:
- removed D2: LED_GREEN_3V3, LED_SMD:LED_1206_3216Metric, symbol Device:LED
- removed R22: 470, Resistor_SMD:R_0805_2012Metric, symbol Device:R
Changed lines of the file:
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@@
   (junction (at 81.28 50.8) (diameter 0) (color 0 0 0 0)
-  )
-  (junction (at 92.71 50.8) (diameter 0) (color 0 0 0 0)
-  )
-  (junction (at 104.14 36.83) (diameter 0) (color 0 0 0 0)
   )
   (junction (at 71.12 36.83) (diameter 0) (color 0 0 0 0)
   )
   (junction (at 59.69 36.83) (diameter 0) (color 0 0 0 0)
-  )
-  (wire (pts (xy 104.14 57.15) (xy 104.14 58.42))
-    (stroke (width 0) (type default) (color 0 0 0 0))
   )
   (wire (pts (xy 81.28 46.99) (xy 81.28 50.8))
@@
     (stroke (width 0) (type default) (color 0 0 0 0))
   )
-  (wire (pts (xy 104.14 58.42) (xy 92.71 58.42))
-    (stroke (width 0) (type default) (color 0 0 0 0))
-  )
   (polyline (pts (xy 165.1 62.23) (xy 39.37 62.23))
     (stroke (width 0) (type default) (color 0 0 0 0))
   )
   (wire (pts (xy 59.69 36.83) (xy 71.12 36.83))
-    (stroke (width 0) (type default) (color 0 0 0 0))
-  )
-  (wire (pts (xy 92.71 50.8) (xy 92.71 58.42))
     (stroke (width 0) (type default) (color 0 0 0 0))
   )
@@
     (stroke (width 0) (type default) (color 0 0 0 0))
   )
-  (wire (pts (xy 104.14 36.83) (xy 107.95 36.83))
-    (stroke (width 0) (type default) (color 0 0 0 0))
-  )
-  (wire (pts (xy 92.71 36.83) (xy 104.14 36.83))
+  (wire (pts (xy 92.71 36.83) (xy 107.95 36.83))
     (stroke (width 0) (type default) (color 0 0 0 0))
   )
@@
     (stroke (width 0) (type default) (color 0 0 0 0))
   )
-  (wire (pts (xy 104.14 48.26) (xy 104.14 49.53))
-    (stroke (width 0) (type default) (color 0 0 0 0))
-  )
   (wire (pts (xy 92.71 36.83) (xy 92.71 39.37))
-    (stroke (width 0) (type default) (color 0 0 0 0))
-  )
-  (wire (pts (xy 104.14 36.83) (xy 104.14 40.64))
     (stroke (width 0) (type default) (color 0 0 0 0))
   )
@@
     )
   )
-  (symbol (lib_id "Device:LED") (at 104.14 53.34 90) (unit 1)
-    (in_bom yes) (on_board yes) (fields_autoplaced)
-    (property "Reference" "D2" (id 0) (at 107.061 54.0928 90)
-      (effects (font (size 1.27 1.27)) (justify right))
-    )
-    (property "Value" "LED_GREEN_3V3" (id 1) (at 107.061 56.6297 90)
-      (effects (font (size 1.27 1.27)) (justify right))
-    )
-    (property "Footprint" "LED_SMD:LED_1206_3216Metric" (id 2) (at 104.14 53.34 0)
-      (effects (font (size 1.27 1.27)) hide)
-    )
-    (property "Datasheet" "~" (id 3) (at 104.14 53.34 0)
-      (effects (font (size 1.27 1.27)) hide)
-    )
-    (pin "1")
-    (pin "2")
-  )
   (symbol (lib_id "Device:C") (at 59.69 43.18 0) (unit 1)
     (in_bom yes) (on_board yes)
@@
       (effects (font (size 1.27 1.27)) hide)
     )
-    (pin "1")
-    (pin "2")
-  )
-  (symbol (lib_id "Device:R") (at 104.14 44.45 0) (unit 1)
-    (in_bom yes) (on_board yes)
-    (property "Reference" "R22" (id 0) (at 105.918 43.2816 0)
-      (effects (font (size 1.27 1.27)) (justify left))
-    )
-    (property "Value" "470" (id 1) (at 105.918 45.593 0)
-      (effects (font (size 1.27 1.27)) (justify left))
-    )
-    (property "Footprint" "Resistor_SMD:R_0805_2012Metric" (id 2) (at 102.362 44.45 90)
-      (effects (font (size 1.27 1.27)) hide)
-    )
-    (property "Datasheet" "~" (id 3) (at 104.14 44.45 0)
-      (effects (font (size 1.27 1.27)) hide)
-    )
