File: Layblar_PCB.kicad_pcb (KiCad board)
At the start: 4 copper layers, 37.3 x 70.3 mm, 36 parts, among them J1 6P6C, J2 USB_C_Receptacle_USB2.0, SW1 SW_Push, SW2 SW_Push, U1 ESP32-C3-MINI-1, U5 NCN5150DG, U8 SE5218

Commit message: Created Version 1.0
Refactored board with tipps after coaching
Parts:
- removed D2: LED_GREEN_3V3, LED_SMD:LED_1206_3216Metric
- removed R22: 470, Resistor_SMD:R_0805_2012Metric
- added C7: 100u, Capacitor_SMD:CP_Elec_6.3x7.7, F.Cu at (55.8, 42.5)
- R4: value 30k -> 4k
- moved C10 4.75 mm to (55.1, 32.2)
- moved C28 4.75 mm to (59.0, 32.2)
- moved U8 4.75 mm to (57.1, 35.5)
Connections:
- U5 pad 3: unconnected-(U5-Pad3) -> Net-(U5-Pad3)
Routing:
- net Net-(U5-Pad3): track 0.00 -> 23.3 mm
- net +3.3V: track 55.7 -> 51.9 mm
- net GND: track 21.0 -> 24.8 mm, vias 2 -> 4
- net +5V: track 16.3 -> 12.8 mm
- net Net-(D2-Pad2): track 3.25 -> 0.00 mm
- net RX_ESP32: track 59.7 -> 57.4 mm
- net TX_ESP32: track 56.3 -> 57.4 mm

Commit message: Updated docs and fixed bug
Connections:
- U1 pad 18: TX_ESP32 -> unconnected-(U1-Pad18)
- U5 pad 11: +3.3V -> unconnected-(U5-Pad11)
- U5 pad 13: TX_ESP32 -> unconnected-(U5-Pad13)
Routing:
- net TX_ESP32: track 57.4 -> 0.00 mm
- net +3.3V: track 51.9 -> 48.8 mm
Changed lines of the file:
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@@
   (net 18 "GPIO_LED_BLUE")
   (net 19 "Net-(D3-Pad2)")
-  (net 20 "Net-(U5-Pad3)")
+  (net 20 "Net-(C7-Pad1)")
   (net 21 "EN")
   (net 22 "GPIO_LED_YELLOW")
@@
   (net 56 "unconnected-(U1-Pad13)")
   (net 57 "unconnected-(U1-Pad16)")
-  (net 58 "TX_ESP32")
-  (net 59 "RX_ESP32")
-  (net 60 "unconnected-(U1-Pad30)")
-  (net 61 "unconnected-(U1-Pad31)")
+  (net 58 "RX_ESP32")
+  (net 59 "unconnected-(U1-Pad30)")
+  (net 60 "unconnected-(U1-Pad31)")
+  (net 61 "unconnected-(U5-Pad11)")
+  (net 62 "unconnected-(U1-Pad18)")
+  (net 63 "unconnected-(U5-Pad13)")
   (footprint "Resistor_SMD:R_0805_2012Metric" (layer "F.Cu")
     (at 55.2625 51.25)
@@
     (fp_circle (center 0 0) (end 3.15 0) (layer "F.Fab") (width 0.1) (fill none))
     (pad "1" smd roundrect (at -2.7 0) (size 3.5 1.6) (layers "F.Cu" "F.Paste" "F.Mask") (roundrect_rratio 0.15625)
-      (net 20 "Net-(U5-Pad3)") (pintype "passive"))
+      (net 20 "Net-(C7-Pad1)") (pintype "passive"))
     (pad "2" smd roundrect (at 2.7 0) (size 3.5 1.6) (layers "F.Cu" "F.Paste" "F.Mask") (roundrect_rratio 0.15625)
       (net 1 "GND") (pintype "passive"))
@@
       (net 46 "unconnected-(U5-Pad2)") (pinfunction "VB") (pintype "power_in"))
     (pad "3" smd rect locked (at -2.725 -1.905 90) (size 0.65 1.55) (layers "F.Cu" "F.Paste" "F.Mask")
-      (net 20 "Net-(U5-Pad3)") (pinfunction "STC") (pintype "output"))
+      (net 20 "Net-(C7-Pad1)") (pinfunction "STC") (pintype "output"))
     (pad "4" smd rect locked (at -2.725 -0.635 90) (size 0.65 1.55) (layers "F.Cu" "F.Paste" "F.Mask")
       (net 45 "Net-(R4-Pad2)") (pinfunction "RIDD") (pintype "input"))
@@
       (net 50 "unconnected-(U5-Pad7)") (pinfunction "TXI") (pintype "output"))
     (pad "8" smd rect locked (at -2.725 4.445 90) (size 0.65 1.55) (layers "F.Cu" "F.Paste" "F.Mask")
-      (net 59 "RX_ESP32") (pinfunction "TX") (pintype "output"))
+      (net 58 "RX_ESP32") (pinfunction "TX") (pintype "output"))
     (pad "9" smd rect locked (at 2.725 4.445 90) (size 0.65 1.55) (layers "F.Cu" "F.Paste" "F.Mask")
       (net 14 "+3.3V") (pinfunction "VIO") (pintype "input"))
@@
       (net 53 "unconnected-(U5-Pad10)") (pinfunction "VS") (pintype "output"))
     (pad "11" smd rect locked (at 2.725 1.905 90) (size 0.65 1.55) (layers "F.Cu" "F.Paste" "F.Mask")
-      (net 14 "+3.3V") (pinfunction "VDD") (pintype "power_in"))
+      (net 61 "unconnected-(U5-Pad11)") (pinfunction "VDD") (pintype "power_in"))
     (pad "12" smd rect locked (at 2.725 0.635 90) (size 0.65 1.55) (layers "F.Cu" "F.Paste" "F.Mask")
       (net 55 "unconnected-(U5-Pad12)") (pinfunction "RX") (pintype "input"))
     (pad "13" smd rect locked (at 2.725 -0.635 90) (size 0.65 1.55) (layers "F.Cu" "F.Paste" "F.Mask")
-      (net 58 "TX_ESP32") (pinfunction "RXI") (pintype "input"))
+      (net 63 "unconnected-(U5-Pad13)") (pinfunction "RXI") (pintype "input"))
     (pad "14" smd rect locked (at 2.725 -1.905 90) (size 0.65 1.55) (layers "F.Cu" "F.Paste" "F.Mask")
       (net 51 "Net-(R11-Pad2)") (pinfunction "RIS") (pintype "input"))
@@
       (net 35 "unconnected-(U1-Pad17)") (pinfunction "NC") (pintype "no_connect"))
     (pad "18" smd rect (at 0 7.6 180) (size 0.4 0.8) (layers "F.Cu" "F.Paste" "F.Mask")
-      (net 58 "TX_ESP32") (pinfunction "GPIO4/ADC1_CH4") (pintype "bidirectional"))
+      (net 62 "unconnected-(U1-Pad18)") (pinfunction "GPIO4/ADC1_CH4") (pintype "bidirectional"))
     (pad "19" smd rect (at 0.8 7.6 180) (size 0.4 0.8) (layers "F.Cu" "F.Paste" "F.Mask")
-      (net 59 "RX_ESP32") (pinfunction "GPIO5/ADC2_CH0") (pintype "bidirectional"))
+      (net 58 "RX_ESP32") (pinfunction "GPIO5/ADC2_CH0") (pintype "bidirectional"))
     (pad "20" smd rect (at 1.6 7.6 180) (size 0.4 0.8) (layers "F.Cu" "F.Paste" "F.Mask")
       (net 22 "GPIO_LED_YELLOW") (pinfunction "GPIO6") (pintype "bidirectional"))
@@
       (net 40 "unconnected-(U1-Pad29)") (pinfunction "NC") (pintype "no_connect"))
     (pad "30" smd rect (at 5.9 2.7 270) (size 0.4 0.8) (layers "F.Cu" "F.Paste" "F.Mask")
-      (net 60 "unconnected-(U1-Pad30)") (pinfunction "GPIO20/U0RXD") (pintype "bidirectional"))
+      (net 59 "unconnected-(U1-Pad30)") (pinfunction "GPIO20/U0RXD") (pintype "bidirectional"))
     (pad "31" smd rect (at 5.9 1.9 270) (size 0.4 0.8) (layers "F.Cu" "F.Paste" "F.Mask")
-      (net 61 "unconnected-(U1-Pad31)") (pinfunction "GPIO21/U0TXD") (pintype "bidirectional"))
+      (net 60 "unconnected-(U1-Pad31)") (pinfunction "GPIO21/U0TXD") (pintype "bidirectional"))
     (pad "32" smd rect (at 5.9 1.1 270) (size 0.4 0.8) (layers "F.Cu" "F.Paste" "F.Mask")
       (net 41 "unconnected-(U1-Pad32)") (pinfunction "NC") (pintype "no_connect"))
@@
   (segment (start 58.95 66.75) (end 59 66.8) (width 0.4) (layer "F.Cu") (net 14))
   (segment (start 62 66.8) (end 62 69.3) (width 0.4) (layer "F.Cu") (net 14))
-  (segment (start 40.7875 41.03) (end 41.78 41.03) (width 0.4) (layer "F.Cu") (net 14))
   (segment (start 34.25 49.25) (end 32.75 50.75) (width 0.4) (layer "F.Cu") (net 14))
   (segment (start 54.35 55.425) (end 54.275 55.5) (width 0.4) (layer "F.Cu") (net 14))
@@
   (segment (start 56.75 66.75) (end 58.95 66.75) (width 0.4) (layer "F.Cu") (net 14))
   (segment (start 59 66.8) (end 62 66.8) (width 0.4) (layer "F.Cu") (net 14))
-  (segment (start 41.78 41.03) (end 43.25 42.5) (width 0.4) (layer "F.Cu") (net 14))
   (segment (start 58.5 70.625) (end 59 71.125) (width 0.3) (layer "F.Cu") (net 14))
   (segment (start 40.5 49.25) (end 36.55 49.25) (width 0.4) (layer "F.Cu") (net 14))
@@
   (segment (start 45.43 37.22) (end 40.7875 37.22) (width 0.4) (layer "F.Cu") (net 51))
   (segment (start 45.5375 37.1125) (end 45.43 37.22) (width 0.4) (layer "F.Cu") (net 51))
-  (segment (start 47.475 62.4) (end 55.165686 62.4) (width 0.2) (layer "F.Cu") (net 58))
-  (segment (start 62.081372 58.55) (end 63.875 56.756371) (width 0.2) (layer "F.Cu") (net 58))
-  (segment (start 55.165686 62.4) (end 59.015686 58.55) (width 0.2) (layer "F.Cu") (net 58))
-  (segment (start 59.015686 58.55) (end 62.081372 58.55) (width 0.2) (layer "F.Cu") (net 58))
-  (segment (start 63.875 56.756371) (end 63.875 45.097183) (width 0.2) (layer "F.Cu") (net 58))
-  (segment (start 46.95 62.925) (end 47.475 62.4) (width 0.2) (layer "F.Cu") (net 58))
-  (segment (start 57.267817 38.49) (end 40.7875 38.49) (width 0.2) (layer "F.Cu") (net 58))
-  (segment (start 63.875 45.097183) (end 57.267817 38.49) (width 0.2) (layer "F.Cu") (net 58))
-  (segment (start 46.95 63.325) (end 46.95 62.925) (width 0.2) (layer "F.Cu") (net 58))
-  (segment (start 63.475 56.590686) (end 63.475 50.847183) (width 0.2) (layer "F.Cu") (net 59))
-  (segment (start 57.422817 44.795) (end 36.5625 44.795) (width 0.2) (layer "F.Cu") (net 59))
-  (segment (start 58.85 58.15) (end 61.915686 58.15) (width 0.2) (layer "F.Cu") (net 59))
-  (segment (start 55 62) (end 58.85 58.15) (width 0.2) (layer "F.Cu") (net 59))
-  (segment (start 46.15 62.6) (end 46.75 62) (width 0.2) (layer "F.Cu") (net 59))
-  (segment (start 46.75 62) (end 55 62) (width 0.2) (layer "F.Cu") (net 59))
-  (segment (start 46.15 63.325) (end 46.15 62.6) (width 0.2) (layer "F.Cu") (net 59))
-  (segment (start 63.475 50.847183) (end 57.422817 44.795) (width 0.2) (layer "F.Cu") (net 59))
-  (segment (start 61.915686 58.15) (end 63.475 56.590686) (width 0.2) (layer "F.Cu") (net 59))
-  (segment (start 36.5625 44.795) (end 35.3375 43.57) (width 0.2) (layer "F.Cu") (net 59))
+  (segment (start 63.475 56.590686) (end 63.475 50.847183) (width 0.2) (layer "F.Cu") (net 58))
+  (segment (start 57.422817 44.795) (end 36.5625 44.795) (width 0.2) (layer "F.Cu") (net 58))
+  (segment (start 58.85 58.15) (end 61.915686 58.15) (width 0.2) (layer "F.Cu") (net 58))
+  (segment (start 55 62) (end 58.85 58.15) (width 0.2) (layer "F.Cu") (net 58))
+  (segment (start 46.15 62.6) (end 46.75 62) (width 0.2) (layer "F.Cu") (net 58))
+  (segment (start 46.75 62) (end 55 62) (width 0.2) (layer "F.Cu") (net 58))
+  (segment (start 46.15 63.325) (end 46.15 62.6) (width 0.2) (layer "F.Cu") (net 58))
+  (segment (start 63.475 50.847183) (end 57.422817 44.795) (width 0.2) (layer "F.Cu") (net 58))
+  (segment (start 61.915686 58.15) (end 63.475 56.590686) (width 0.2) (layer "F.Cu") (net 58))
+  (segment (start 36.5625 44.795) (end 35.3375 43.57) (width 0.2) (layer "F.Cu") (net 58))
   (zone (net 1) (net_name "GND") (layer "F.Cu") (hatch edge 0.508)
     (connect_pads (clearance 0.508))

Commit message: Updated R4 Value and docs
Parts:
- R4: value 4k -> 13k
Changed lines of the file:
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@@
       (effects (font (size 1 1) (thickness 0.15)))
     )
-    (fp_text value "4k" (at 0 1.65 90) (layer "F.Fab")
+    (fp_text value "13k" (at 0 1.65 90) (layer "F.Fab")
       (effects (font (size 1 1) (thickness 0.15)))
     )
