File: Layblar_PCB.kicad_sch (KiCad schematic)
At the start: 23 parts, among them J2 USB_C_Receptacle_USB2.0, SW1 SW_Push, SW2 SW_Push, U1 ESP32-C3-MINI-1

Commit message: Updated docs and fixed bug
Connections:
- net TX_ESP32: no longer names the net of U1.18 (GPIO4/ADC1_CH4)
Changed lines of the file:
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@@
-    (stroke (width 0) (type default) (color 0 0 0 0))
-  )
-  (wire (pts (xy 175.26 83.82) (xy 194.31 83.82))
     (stroke (width 0) (type default) (color 0 0 0 0))
   )
@@
       (effects (font (size 1.27 1.27)) (justify left) hide)
     )
-  )
-  (global_label "TX_ESP32" (shape input) (at 194.31 83.82 0) (fields_autoplaced)
-    (effects (font (size 1.27 1.27)) (justify left))
-    (property "Intersheet References" "${INTERSHEET_REFS}" (id 0) (at 205.8266 83.7406 0)
-      (effects (font (size 1.27 1.27)) (justify left) hide)
-    )
